File: hw/zumo_tb_01.brd (EAGLE design)
At the start: 99.1 x 91.4 mm, 156 parts, among them IC1 LT 1963 AEST-3.3 (1.5A), IC10 ESP32-WROVER, IC11 MCP1703DB, IC12 MCP1703DB, IC2 MCP1703DB, IC3 LM317MBSTT3, IC5 STM32G081RBT6, K1 68712414522, Q1 IRLML5203, Q2 BSS138, Q3 BSS138, U1 W25Q40BVSN

Commit message: -
Parts:
- added SJ26: (no value), jumper:SJ
Connections:
- net U5: now also SJ26.1
- net ZUMO_5V: now also SJ26.2
Routing:
- net U5: track 216.3 -> 228.7 mm, vias 15 -> 17
- net ZUMO_5V: track 17.0 -> 20.6 mm, vias 0 -> 1
- net INT: track 151.1 -> 152.8 mm
- net N$10: track 65.6 -> 66.2 mm
- net GND: vias 96 -> 97
- added copper zone on layer 1, net N$10
- added copper zone on layer 16, net N$11
- added copper zone on layer 1, net U_CHARGE1
- added copper zone on layer 16, net U_CHARGE1
- added copper zone on layer 1, net U_CHARGE2
- added copper zone on layer 16, net U_CHARGE2
Other:
- board text added: "ZUMO 32U4 ESP32/OPI/RPI Shield V1.2"
- board text removed: "ZUMO 32U4 ESP32/OPI/RPI Shield V1.0"
