File: hw/zumo_tb_01.sch (EAGLE design)
At the start: 156 parts, among them IC1 LT 1963 AEST-3.3 (1.5A), IC10 ESP32-WROVER, IC11 MCP1703DB, IC12 MCP1703DB, IC2 MCP1703DB, IC3 LM317MBSTT3, IC5 STM32G081RBT6, K1 68712414522, Q1 IRLML5203, Q2 BSS138, Q3 BSS138, U1 W25Q40BVSN

Commit message: -
Parts:
- added SJ26: (no value), jumper:SJ
Connections:
- net U5: now also SJ26.1
- net ZUMO_5V: now also SJ26.2
Changed lines of the file:
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@@
 <part name="R11" library="rcl" library_urn="urn:adsk.eagle:library:334" deviceset="R-EU_" device="R0603" package3d_urn="urn:adsk.eagle:package:23555/3"/>
 <part name="SJ23" library="jumper" library_urn="urn:adsk.eagle:library:252" deviceset="SJ" device="" package3d_urn="urn:adsk.eagle:package:15471/1"/>
+<part name="SJ26" library="jumper" library_urn="urn:adsk.eagle:library:252" deviceset="SJ" device="" package3d_urn="urn:adsk.eagle:package:15471/1"/>
 </parts>
 <sheets>
@@
 <attribute name="VALUE" x="112.522" y="214.63" size="1.778" layer="96" rot="R90"/>
 </instance>
+<instance part="SJ26" gate="1" x="78.74" y="233.68" smashed="yes" rot="R270">
+<attribute name="NAME" x="81.28" y="236.22" size="1.778" layer="95" rot="R270"/>
+<attribute name="VALUE" x="74.93" y="236.22" size="1.778" layer="96" rot="R270"/>
+</instance>
 </instances>
 <busses>
@@
 <wire x1="157.48" y1="20.32" x2="154.94" y2="20.32" width="0.1524" layer="91"/>
 <label x="154.94" y="20.32" size="1.016" layer="95" rot="R180" xref="yes"/>
+</segment>
+<segment>
+<pinref part="SJ26" gate="1" pin="1"/>
+<wire x1="78.74" y1="238.76" x2="78.74" y2="241.3" width="0.1524" layer="91"/>
+<label x="78.74" y="241.3" size="1.016" layer="95" rot="R90" xref="yes"/>
 </segment>
 </net>
@@
 <pinref part="SV7" gate="G$1" pin="4"/>
 </segment>
-</net>
+<segment>
+<pinref part="SJ26" gate="1" pin="2"/>
+<wire x1="78.74" y1="228.6" x2="78.74" y2="226.06" width="0.1524" layer="91"/>
+<label x="78.74" y="226.06" size="1.016" layer="95" rot="R270" xref="yes"/>
+</segment>
+</net>
